Commit message: optimizer_finished

File: demo_ws/install/cpp_bs_demo/share/cpp_bs_demo/urdf/ball_obstacle.urdf (robot description, URDF)
Before this commit: robot ball_obstacle, 2 links, 1 joints
Joints:
- joint base_to_ball: origin xyz=1 1 1 rpy=0 0 0 -> xyz=4 2 2 rpy=0 0 0

Commit message: demo finished

File: demo_ws/install/cpp_bs_demo/share/cpp_bs_demo/urdf/ball_obstacle.urdf (robot description, URDF)
Before this commit: robot ball_obstacle, 2 links, 1 joints
Joints:
- joint base_to_ball: origin xyz=4 2 2 rpy=0 0 0 -> xyz=0 0 0 rpy=0 0 0
